File: ECU_BOARD.kicad_pcb (KiCad board)
At the start: 2 copper layers, 71 x 101.6 mm, 17 parts, among them Q1 RFP30N06LE, Q2 RFP30N06LE, U1 Teensy4.0

Commit message: finished
Parts:
- added VReg1: B04B-XASK-1(LF)(SN), Connector_PinSocket_2.54mm:PinSocket_1x04_P2.54mm_Vertical, F.Cu at (142.2, 95.7)
- moved R3 127.9 mm to (156.8, 137.6), turned to -90 degrees
- moved R1 124.1 mm to (156.8, 124.3), turned to -90 degrees
- moved Q2 123.8 mm to (145.3, 137.2), turned to 90 degrees
- moved R4 121.4 mm to (151.8, 127.4), turned to -90 degrees
- moved R2 110.1 mm to (151.8, 114.2), turned to -90 degrees
- moved R5 105.6 mm to (149.5, 100.9), turned to 180 degrees
- moved TP1 96.1 mm to (153.8, 107.7)
- moved D2 95.2 mm to (131.4, 145.4)
- moved TP3 95.1 mm to (153.8, 96.2)
- moved TP2 95.1 mm to (153.8, 101.9)
- moved D1 85.9 mm to (131.3, 110.2)
- moved CANMotor1 67.7 mm to (155.7, 67.3), turned to 0 degrees
- moved CANData1 67.7 mm to (171.0, 67.3), turned to 0 degrees
- moved 6P_ECU1 43.7 mm to (125.4, 81.8)
- moved H_BL1 43.7 mm to (126.0, 123.2)
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Connections:
- Q1 pad 1: /HORN IN -> Net-(Q1-G)
- Q1 pad 2: (no net) -> /HORN IN
Routing:
- net /12V: track 0.00 -> 118.3 mm
- net /5V: track 0.00 -> 92.5 mm
- net /3.3V: track 0.00 -> 91.5 mm
- net /CANL_D: track 0.00 -> 63.1 mm
- net /CANH_D: track 0.00 -> 56.8 mm
- net /BL IN: track 0.00 -> 56.1 mm
- net /CANH_M: track 0.00 -> 47.9 mm
- net /CRX11: track 0.00 -> 38.1 mm
- net /D3: track 0.00 -> 34.8 mm
- net /CANL_M: track 0.00 -> 34.6 mm
- net /CTX11: track 0.00 -> 34.2 mm
- net /CTX21: track 0.00 -> 30.8 mm
- net /HORN IN: track 0.00 -> 26.6 mm
- net /CRX21: track 0.00 -> 25.8 mm
- net /D2: track 0.00 -> 18.0 mm
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- added copper zone on F.Cu, net GND
