File: ECU_BOARD.kicad_sch (KiCad schematic)
At the start: 18 parts, among them Q1 RFP30N06LE, Q2 RFP30N06LE, U1 Teensy4.0

Commit message: finished
Parts:
- VReg1: footprint Connector_PinSocket_2.54mm:PinSocket_1x04_P2.54mm_Horizontal -> Connector_PinSocket_2.54mm:PinSocket_1x04_P2.54mm_Vertical
Connections:
- net HORN IN: now also Q1.2 (D); no longer Q1.1 (D)
Changed lines of the file:
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@@
 	(wire
 		(pts
+			(xy 173.99 133.35) (xy 173.99 132.08)
+		)
+		(stroke
+			(width 0)
+			(type default)
+		)
+	)
+	(wire
+		(pts
 			(xy 229.87 107.95) (xy 234.95 107.95)
 		)
@@
 	(wire
 		(pts
-			(xy 187.96 91.44) (xy 187.96 93.98)
+			(xy 187.96 91.44) (xy 187.96 97.79)
 		)
 		(stroke
@@
 		(pin "1"
 		)
-		(pin "1"
+		(pin "2"
 		)
 		(instances
@@
 	(symbol
 		(lib_id "ECU_BOARD-altium-import:GND_POWER_GROUND")
-		(at 173.99 132.08 0)
+		(at 173.99 133.35 0)
 		(unit 1)
 		(exclude_from_sim no)
@@
 		(dnp no)
 		(property "Reference" "#PWR0102"
-			(at 173.99 132.08 0)
+			(at 173.99 133.35 0)
 			(effects
 				(font
@@
 		)
 		(property "Value" "GND"
-			(at 173.99 138.43 0)
+			(at 173.99 139.7 0)
 			(effects
 				(font
@@
 		)
 		(property "Footprint" ""
-			(at 173.99 132.08 0)
+			(at 173.99 133.35 0)
 			(effects
 				(font
@@
 		)
 		(property "Datasheet" ""
-			(at 173.99 132.08 0)
+			(at 173.99 133.35 0)
 			(effects
 				(font
@@
 		)
 		(property "Description" ""
-			(at 173.99 132.08 0)
+			(at 173.99 133.35 0)
 			(effects
 				(font
@@
 	(symbol
 		(lib_id "ECU_BOARD-altium-import:GND_POWER_GROUND")
-		(at 187.96 93.98 0)
+		(at 187.96 97.79 0)
 		(unit 1)
 		(exclude_from_sim no)
@@
 		(dnp no)
 		(property "Reference" "#PWR0107"
-			(at 187.96 93.98 0)
+			(at 187.96 97.79 0)
 			(effects
 				(font
@@
 		)
 		(property "Value" "GND"
-			(at 187.96 100.33 0)
+			(at 187.96 104.14 0)
 			(effects
 				(font
@@
 		)
 		(property "Footprint" ""
-			(at 187.96 93.98 0)
+			(at 187.96 97.79 0)
 			(effects
 				(font
@@
 		)
 		(property "Datasheet" ""
-			(at 187.96 93.98 0)
+			(at 187.96 97.79 0)
 			(effects
 				(font
@@
 		)
 		(property "Description" ""
-			(at 187.96 93.98 0)
+			(at 187.96 97.79 0)
 			(effects
 				(font
@@
 			)
 		)
-		(property "Footprint" "Connector_PinSocket_2.54mm:PinSocket_1x04_P2.54mm_Horizontal"
+		(property "Footprint" "Connector_PinSocket_2.54mm:PinSocket_1x04_P2.54mm_Vertical"
 			(at 187.96 36.83 0)
 			(effects
